Commit message: backup

File: littlebot/urdf/little_bot.urdf (robot description, URDF)
Before this commit: robot little_bot, 11 links, 10 joints
Links:
- removed link z_rail_link-v1
- removed link z_slider_link-v1
- added link z_rail_link-v5, mass 0.31575562187676676; collision mesh filename=package://littlebot/meshes/z_rail_link-v5.stl scale=0.001 0.001 0.001; visual mesh filename=package://littlebot/meshes/z_rail_link-v5.stl scale=0.001 0.001 0.001
- added link z_slider_link-v5, mass 0.031761577565023694; collision mesh filename=package://littlebot/meshes/z_slider_link-v5.stl scale=0.001 0.001 0.001; visual mesh filename=package://littlebot/meshes/z_slider_link-v5.stl scale=0.001 0.001 0.001
- link arm_link-v1: geometry collision mesh filename=package://littlebot/meshes/arm_link-v1.stl scale=0.001 0.001 0.001; visual mesh filename=package://littlebot/meshes/arm_link-v1.stl scale=0.001 0.001 0.001
Joints:
- removed joint z_rail_link-v1_camera_joint
- removed joint z_rail_link-v1_z_axis_joint
- removed joint z_slider_link-v1_arm_joint
- added joint z_rail_link-v5_camera_joint: type fixed, parent z_rail_link-v5, child camera-v1, origin xyz=0.024748739999999998 0.024748739999999998 0.125 rpy=-9.860761315262648e-32 -0.0 -5.153823899991262e-47
- added joint z_rail_link-v5_z_axis_joint: type prismatic, parent z_rail_link-v5, child z_slider_link-v5, origin xyz=0.024748739999999998 0.024748739999999998 0.005 rpy=-9.860761315262648e-32 -0.0 -5.153823899991262e-47, axis 0.0 -9.860761315262648e-32 1.0, limit lower=0.0 upper=0.095 effort=1000000 velocity=1000000
- added joint z_slider_link-v5_arm_joint: type continuous, parent z_slider_link-v5, child arm_link-v1, origin xyz=0.153 -0.015 0.105 rpy=1.5707963267948966 0.0 0.0, axis 0.0 0.0 -1.0
- joint base_link_front_left_wheel_joint: axis 0.0 0.0 1.0 -> (none); origin xyz=0.07 0.13 0.0125 rpy=-1.5707963267948966 -0.0 0.0 -> xyz=0.07 0.128 0.0125 rpy=0 0 0
- joint base_link_front_right_wheel_joint: axis 0.0 0.0 1.0 -> (none); origin xyz=0.07 -0.13 0.0125 rpy=1.5707963267948966 -0.0 0.0 -> xyz=0.07 -0.128 0.0125 rpy=0 0 0
- joint base_link_pillar_fixed_joint: child z_rail_link-v1 -> z_rail_link-v5; origin xyz=-0.01775126 -0.024748739999999998 0.07 rpy=0.0 -0.0 0.0 -> xyz=-0.06724874 -0.024748739999999998 0.07 rpy=0.0 -0.0 0.0
- joint base_link_rear_left_wheel_joint: axis 0.0 0.0 1.0 -> (none); origin xyz=-0.07 0.13 0.0125 rpy=-1.5707963267948966 -0.0 0.0 -> xyz=-0.07 0.128 0.0125 rpy=0 0 0
- joint base_link_rear_right_wheel_joint: axis 0.0 0.0 1.0 -> (none); origin xyz=-0.07 -0.13 0.0125 rpy=1.5707963267948966 -0.0 0.0 -> xyz=-0.07 -0.128 0.0125 rpy=0 0 0

Commit message: back to ver1

File: littlebot/urdf/little_bot.urdf (robot description, URDF)
Before this commit: robot little_bot, 11 links, 10 joints
Links:
- removed link z_rail_link-v5
- removed link z_slider_link-v5
- added link z_rail_link-v1, mass 0.2; collision box size=0.026 0.026 0.09; collision mesh filename=package://littlebot/meshes/z_rail_link-v1.stl scale=0.001 0.001 0.001
- added link z_slider_link-v1, mass 0.1; collision box size=0.020 0.020 0.090; collision mesh filename=package://littlebot/meshes/z_slider_link-v1.stl scale=0.001 0.001 0.001
- link arm_link-v1: mass 0.03346092824173876 -> 0.1
- link base_link: mass 1.214879905211409 -> 1.514879905211409
Joints:
- removed joint z_rail_link-v5_camera_joint
- removed joint z_rail_link-v5_z_axis_joint
- removed joint z_slider_link-v5_arm_joint
- added joint z_rail_link-v1_camera_joint: type fixed, parent z_rail_link-v1, child camera-v1, origin xyz=-0.024748739999999998 0.024748739999999998 0.105 rpy=7.888609052210118e-31 -0.0 0.0
- added joint z_rail_link-v1_z_axis_joint: type prismatic, parent z_rail_link-v1, child z_slider_link-v1, origin xyz=-0.03474874 0.03474874 0.01 rpy=7.888609052210118e-31 -0.0 0.0, axis 0.0 0.0 1.0, limit lower=-0.03 upper=0.03 effort=20.0 velocity=0.2
- added joint z_slider_link-v1_arm_joint: type revolute, parent z_slider_link-v1, child arm_link-v1, origin xyz=0.1275 0.0052499999999999995 0.05900625000000001 rpy=1.5707963267948966 -0.0 0.0, axis 0.0 0.0 1.0, limit lower=-0.8 upper=0.8 effort=8.0 velocity=0.2
- joint base_link_front_left_wheel_joint: origin xyz=0.07 0.128 0.0125 rpy=0 0 0 -> xyz=0.07 0.13 0.0125 rpy=-1.5707963267948966 -0.0 0.0
- joint base_link_front_right_wheel_joint: origin xyz=0.07 -0.128 0.0125 rpy=0 0 0 -> xyz=0.07 -0.13 0.0125 rpy=1.5707963267948966 -0.0 0.0
- joint base_link_pillar_fixed_joint: child z_rail_link-v5 -> z_rail_link-v1; origin xyz=-0.06724874 -0.024748739999999998 0.07 rpy=0.0 -0.0 0.0 -> xyz=-0.01775126 -0.024748739999999998 0.07 rpy=0.0 -0.0 0.0
- joint base_link_rear_left_wheel_joint: origin xyz=-0.07 0.128 0.0125 rpy=0 0 0 -> xyz=-0.07 0.13 0.0125 rpy=-1.5707963267948966 -0.0 0.0
- joint base_link_rear_right_wheel_joint: origin xyz=-0.07 -0.128 0.0125 rpy=0 0 0 -> xyz=-0.07 -0.13 0.0125 rpy=1.5707963267948966 -0.0 0.0

Commit message: da sua duoc loi banh xe va arm_control

File: littlebot/urdf/little_bot.urdf (robot description, URDF)
Before this commit: robot little_bot, 11 links, 10 joints
Joints:
- joint base_link_front_left_wheel_joint: axis (none) -> 0.0 0.0 1.0; type fixed -> continuous
- joint base_link_front_right_wheel_joint: axis (none) -> 0.0 0.0 1.0; type fixed -> continuous
- joint base_link_rear_left_wheel_joint: axis (none) -> 0.0 0.0 1.0; type fixed -> continuous
- joint base_link_rear_right_wheel_joint: axis (none) -> 0.0 0.0 1.0; type fixed -> continuous
- joint z_rail_link-v1_z_axis_joint: limit lower=-0.03 upper=0.03 effort=20.0 velocity=0.2 -> lower=-0.05 upper=0.04 effort=20.0 velocity=0.2
- joint z_slider_link-v1_arm_joint: limit lower=-0.8 upper=0.8 effort=8.0 velocity=0.2 -> lower=-1.0 upper=0.8 effort=8.0 velocity=0.2

Commit message: config imu on rviz and add sample world on gazebo

File: littlebot/urdf/little_bot.urdf (robot description, URDF)
Before this commit: robot little_bot, 11 links, 10 joints
Joints:
- joint base_link_imu_joint: origin xyz=0.0 0.0 0.0 rpy=3.141592653589793 -0.0 0.0 -> xyz=0.0 0.0 0.0 rpy=0.0 0.0 0.0
